File: HapticControl_v0.0/HapticControl.sch (EAGLE design)
At the start: 0 parts

Commit message: initial pcb constraints, and initial sch
Parts:
- added C1, C14, C15, C18, C19, C2, C20, C21, C3, C5, C7, C8: 100n, Passive Components > Capacitors > Multilayer Ceramic Capacitors MLCC:MLCC_0402
- added C10, C9: 3p, Passive Components > Capacitors > Multilayer Ceramic Capacitors MLCC:MLCC_0402
- added C11, C12: (no value), Passive Components > Capacitors > Multilayer Ceramic Capacitors MLCC:MLCC_0402
- added C13, C16, C17: 1u, Passive Components > Capacitors > Multilayer Ceramic Capacitors MLCC:MLCC0603
- added C4: (no value), Passive Components > Capacitors > Multilayer Ceramic Capacitors MLCC:MLCC0603
- added C6: 10u, Passive Components > Capacitors > Multilayer Ceramic Capacitors MLCC:MLCC0603
- added E1: 2.4GHZTRACE-15.2MM, Microstrip Antenna:2.4GHZTRACE-15.2MM
- added L1: 10u, Passive Components > Inductors, Chokes & Coils:INDUCTOR_NC_0805
- added L2: filter, Passive Components > Inductors, Chokes & Coils:INDUCTOR_NC_0603
- added M1: SPH0641LM4H-1, Knowles:SPH0641LM4H-1
- added R1, R2, R4, R5: 100k, Passive Components > Resistors > Chip Resistors:RESISTOR_0402
- added R3, R6: 4k7, Passive Components > Resistors > Chip Resistors:RESISTOR_0402
- added R7, R8, R9: 200k, Passive Components > Resistors > Chip Resistors:RESISTOR_0402
- added TC1: TC2050-IDC, TagConnect:TC2050-IDC
- added TP1, TP2, TP3: TEST_POINT, Utility > Board:TEST_POINT
- added U1: CC2642R, Texas Instruments:CC2642R
- added U2: SST26VF064B, Microchip:SST26VF064B
- added U3: ICM20948, TDK:ICM20948
- added U4: 74LVC1G17, Semiconductors > Integrated Circuits - ICs > Logic ICs > Logic Gates:74LVC1G17
- added U5: MCP1700T-1802TT, Power > LDO Voltage Regulators:MCP1700T-1802TT
- added U6: PCA9306-DCU, Texas Instruments:PCA9306-DCU
- added U7: MTCH6301, Microchip:MTCH6301
- added X1: 48MHz, Crystal:CRYSTAL_4P
- added X2: 32.768kHz, Crystal:CRYSTAL2-SMD-3215
Connections:
- new net 1.8V: C17.P$1, C19.P$1, R8.P$2, R9.P$2, U3.VDDIO, U5.VO, U6.VREF1
- new net 3.3V: C15.P$1, C16.P$1, C18.P$1, L2.P$1, M1.VCC, R2.P$2, R3.P$2, R4.P$2, R5.P$2, R6.P$2, R7.P$2, TC1-1(VTARGET).S, U2.VCC, U3.VDD, U4.PW.GND, U5.VI
- new net DBG_RX: TP2.S, U1.DIO_27
- new net DBG_TX: TP1.S, U1.DIO_28
- new net FLASH_CS: R2.P$1, U1.DIO_30, U2.!CS!
- new net FLASH_MISO: U1.DIO_18, U2.MISO/IO1
- new net FLASH_MOSI: U1.DIO_19, U2.MOSI/IO0
- new net GND: C1.P$2, C10.P$2, C11.P$2, C12.P$2, C13.P$2, C14.P$2, C15.P$2, C16.P$2, C17.P$2, C18.P$2, C19.P$2, C2.P$2, C20.P$2, C21.P$2, C3.P$2, C4.P$2, C5.P$2, C6.P$2, C7.P$2, C8.P$2, C9.P$2, M1.GND, M1.SEL, TC1-3(GND).S, TC1-9(GND).S, TP3.S, U1.GND, U2.GND, U3.GND, U3.SDO, U4.PW.VCC, U5.GND, U6.GND, X1.GND@0, X1.GND@1
- new net I2S_CLK: M1.CLK, U1.DIO_21
- new net I2S_DATIN: M1.DAT, U1.DIO_8
- new net JTAG_TCKC: TC1-4(TCK/SWCLK).S, U1.JTAG_TCKC
- new net JTAG_TDI: TC1-8(TDI).S
- new net JTAG_TDI/FLASH_MOSI: U1.DIO_17, U2.SCK
- new net JTAG_TDO: TC1-6(TDO/SWO).S, U1.DIO_16
- new net JTAG_TMSC: TC1-2(TMS/SWDIO).S, U1.JTAG_TMSC
- new net MCU_!RESET: C14.P$1, R1.P$1, TC1-10(!RESET!).S, U1.!RESET
- new net MCU_SW: L1.P$1, U1.DCDC_SW
- new net MPU_INT: U1.DIO_3, U4.1.Y
- new net N$1: U1.RF_N
- new net N$11: C21.P$1, R7.P$1, U6.EN, U6.VREF2
- new net N$2: C13.P$1, U1.DCOUPL
- new net N$3: U1.RF_P
- new net N$4: U3.INT, U4.1.A
- new net N$5: R8.P$1, U3.SCL, U6.SCL1
- new net N$6: R9.P$1, U3.SDI, U6.SDA1
- new net N$7: R4.P$1, U2.!WP!/IO2
- new net N$8: R5.P$1, U2.!HOLD!/IO3
- new net N$9: C20.P$1, U3.REGOUT
- new net SCL: R6.P$1, U1.DIO_1, U6.SCL2
- new net SDA: R3.P$1, U1.DIO_0, U6.SDA2
- new net VDDR: C6.P$1, C7.P$1, C8.P$1, L1.P$2, U1.VDDR, U1.VDDR_RF
- new net VDDS: C1.P$1, C2.P$1, C3.P$1, C4.P$1, C5.P$1, L2.P$2, R1.P$2, U1.VDDS@0, U1.VDDS@1, U1.VDDS@2, U1.VDDS_DCDC
- new net XTAL_32K_Q1: C10.P$1, U1.X32K_Q1, X2.2
- new net XTAL_32K_Q2: C9.P$1, U1.X32K_Q2, X2.1
- new net XTAL_48M_N: C12.P$1, U1.X48M_N, X1.2
- new net XTAL_48M_P: C11.P$1, U1.X48M_P, X1.1
Other:
- note added: "Pin 13"
- note added: "Pin 22"
- note added: "Pin 34"
- note added: "Pin 44"
- note added: "Pin 45"
- note added: "Pin 48"
- note added: "TODO: Antenna matching"
- note added: "TODO: Buck Converter QI Charger"
- note added: "TODO: Capacitive Buttons Capacitive Matrix Haptic Feedback"
